File: ARSensors/ARSensors.kicad_sch (KiCad schematic)
At the start: 14 parts, among them J1 Conn_01x08, U1 LIS3MDLTR, U2 LSM6DSRTR

Commit message: Add files via upload
Parts:
- removed H3, H4: MountingHole_Pad, MountingHole:MountingHole_4.3mm_M4_Pad_Via, symbol Mechanical:MountingHole_Pad
- removed U1: LIS3MDLTR, LGA-12_2X2X1_STM, symbol 2025-12-07_02-05-02:LIS3MDLTR
- removed U2: LSM6DSRTR, LGA-14L_2P5X3X0P83_STM, symbol 2025-12-07_01-57-28:LSM6DSRTR
- added U2: LIS3MDLTR, footprints1:LGA-12_2X2X1_STM, symbol 2026-01-01_23-09-18:LIS3MDLTR
- added U3: LSM6DSRTR, footprints:LGA-14L_2P5X3X0P83_STM, symbol 2026-01-01_23-09-05:LSM6DSRTR
- C1, C2, C3, C4, C5: footprint (none) -> Capacitor_SMD:C_0402_1005Metric
- J1: footprint (none) -> Connector_PinHeader_2.54mm:PinHeader_1x08_P2.54mm_Vertical
- R1, R2: footprint (none) -> Resistor_SMD:R_0603_1608Metric
Connections:
- net +3.3V: now also U2.10 (CS), U2.5 (VDD), U2.6 (VDD_IO), U3.12 (CS), U3.5 (VDD_IO), U3.8 (VDD)
- net GND: now also U2.12 (RES), U2.2 (RES), U2.3 (GND), U2.9 (SDO/SA1), U3.1 (SDO/SA0), U3.2 (SDX), U3.3 (SCX), U3.6 (GND), U3.7 (GND)
- net I2C1_SCL: now also U2.1 (SCL/SPC), U3.13 (SCL)
- net I2C1_SDA: now also U2.11 (SDA/SDI/SDO), U3.14 (SDA)
- net LIS3MDLTR_DRDY: now also U2.8 (DRDY)
- net LIS3MDLTR_INT: now also U2.7 (INT)
- net LSM6DSR_INT1: now also U3.4 (INT1)
- net LSM6DSR_INT2: now also U3.9 (INT2)
- net at C1.1: now also U2.4 (C1)
