File: ARviewer/ARviewer.kicad_sch (KiCad schematic)
At the start: 63 parts, among them J1 SWD, J2 Display, J3 Sensors, J4 USB_C_Receptacle_USB2.0_16P, SW1 SW_Push, SW2 SW_SPDT, U1 STM32F429VIT6, U2 AP62300TWU-7, U3 USBLC6-2SC6, Y1 25MHz

Commit message: Add files via upload
Parts:
- removed H1, H3: MountingHole_Pad, MountingHole:MountingHole_4.3mm_M4_Pad_Via, symbol Mechanical:MountingHole_Pad
- removed J1: SWD, Connector_PinHeader_2.54mm:PinHeader_2x04_P2.54mm_Vertical, symbol Connector_Generic:Conn_02x04_Odd_Even
- removed J2: Display, Connector_PinSocket_2.54mm:PinSocket_2x18_P2.54mm_Vertical, symbol Connector_Generic:Conn_02x18_Odd_Even
- removed J3: Sensors, Connector_PinHeader_2.54mm:PinHeader_1x08_P2.54mm_Vertical, symbol Connector_Generic:Conn_01x08
- added J1: Conn_01x14, Connector_PinHeader_2.54mm:PinHeader_1x14_P2.54mm_Vertical, symbol Connector_Generic:Conn_01x14
- added J3: Conn_01x19, Connector_PinHeader_2.54mm:PinHeader_1x19_P2.54mm_Vertical, symbol Connector_Generic:Conn_01x19
- added J4: Conn_01x05, Connector_PinHeader_2.54mm:PinHeader_1x05_P2.54mm_Vertical, symbol Connector_Generic:Conn_01x05
- D1, D6: value GREEN -> RED
- D2: value ORANGE -> RED
- D3: value BLUE -> RED
- D4: value YELLOW -> RED
- renumbered H2 to H1, H4 to H2, J4 to J2, R2 to R1, R1 to R10, R3 to R2, R4 to R3, R5 to R4, R6 to R5, R7 to R6, R8 to R7, R9 to R8, R10 to R9
Connections:
- net +3.3V: now also J1.13 (Pin_13), J1.14 (Pin_14)
- net +5V: now also J3.18 (Pin_18), J3.19 (Pin_19)
- net FMC_A16: now also J3.5 (Pin_5)
- net FMC_D0: now also J3.4 (Pin_4)
- net FMC_D1: now also J3.3 (Pin_3)
- net FMC_D10: now also J3.11 (Pin_11)
- net FMC_D11: now also J3.10 (Pin_10)
- net FMC_D12: now also J3.9 (Pin_9)
- net FMC_D13: now also J3.8 (Pin_8)
- net FMC_D14: now also J3.7 (Pin_7)
- net FMC_D15: now also J3.6 (Pin_6)
- net FMC_D2: now also J1.10 (Pin_10)
- net FMC_D3: now also J1.9 (Pin_9)
- net FMC_D4: now also J3.17 (Pin_17)
- net FMC_D5: now also J3.16 (Pin_16)
- net FMC_D6: now also J3.15 (Pin_15)
- net FMC_D7: now also J3.14 (Pin_14)
- net FMC_D8: now also J3.13 (Pin_13)
- net FMC_D9: now also J3.12 (Pin_12)
- net FMC_NE1: now also J1.6 (Pin_6)
- net FMC_NWE: now also J1.7 (Pin_7)
- net FMC_RST: now also J1.8 (Pin_8)
- net GND: now also J1.1 (Pin_1), J1.2 (Pin_2), J3.1 (Pin_1), J3.2 (Pin_2)
- net I2C1_SCL: now also J1.4 (Pin_4)
- net I2C1_SDA: now also J1.3 (Pin_3)
- net LED1: now also U1.32 (PA7); no longer U1.24 (PA1)
- net LIS3MDLTR_DRDY: now also J4.4 (Pin_4)
- net LIS3MDLTR_INT: now also J4.5 (Pin_5)
- net LSM6DSR_INT1: now also J4.3 (Pin_3)
- net LSM6DSR_INT2: now also J4.2 (Pin_2)
- net NRST: now also J4.1 (Pin_1)
- net SYS_JTCK_SWCLK: now also J1.11 (Pin_11)
- net SYS_JTCK_SWO: now also J1.5 (Pin_5)
- net at R10.1: now also J1.12 (Pin_12)
- no-connect marks 57 -> 45
Other:
- note added: "Connectors designed as pinouts due to physical restrictions of chip and 2 layer board. Wanted to minimize traces."
- note added: "Connects Serial Wire Debug"
- note added: "Connects to board containing Accelerometer/Gyroscope (LSM6DSRTR) and Magnetometer (LIS3MDLRTR)"
- note added: "Pin Connectors (Display, Serial Wire Debug, and Sensors)"
- note added: "Pins for 6 bit parallel, FMC & 1 GPIO on STM32CubeMX: https://www.amazon.com/dp/B0D8FL8S9X?ref=ppx_yo2ov_dt_b_fed_asin_title"
- note added: "Rext = 1 / (2 * pi * F * CL2) Rext = 1 / (2 * pi * 25MHz * 14pF) Rext = 454.73 = R3"
- note removed: "16 bit parallel, FMC & 1 GPIO on STM32CubeMX https://www.amazon.com/dp/B0D8FL8S9X?ref=ppx_yo2ov_dt_b_fed_asin_title"
- note removed: "Connector to board containing Accelerometer/Gyroscope (LSM6DSRTR) and Magnetometer (LIS3MDLRTR)"
- note removed: "Display Connector"
- note removed: "Rext = 1 / (2 * pi * F * CL2) Rext = 1 / (2 * pi * 25MHz * 14pF) Rext = 454.73 = R4"
- note removed: "Sensors Connector"
- note removed: "Serial Wire Debug"
- moved on the sheet: H1, H2, R10
